Commit message: Add Lidar to the robot

File: install/robot_description/share/robot_description/urdf/robot.urdf (robot description, URDF)
Before this commit: robot robot, 4 links, 3 joints
Links:
- added link link_laser_scan, mass 0.5; collision cylinder length=0.20 radius=0.15; visual cylinder length=0.20 radius=0.15
Joints:
- added joint joint_laser_scan_chassis: type fixed, parent link_chassis, child link_laser_scan, origin xyz=0.8 0 0.3 rpy=0 0 0

File: src/robot_description/urdf/robot.urdf (robot description, URDF)
Before this commit: robot robot, 4 links, 3 joints
Links:
- added link link_laser_scan, mass 0.5; collision cylinder length=0.20 radius=0.15; visual cylinder length=0.20 radius=0.15
Joints:
- added joint joint_laser_scan_chassis: type fixed, parent link_chassis, child link_laser_scan, origin xyz=0.8 0 0.3 rpy=0 0 0
