Commit message: Summon Multiple robots in Gazebo world

File: install/robot_description/share/robot_description/urdf/robot.xacro (robot description, xacro)
@@ -1,180 +1,183 @@
 <?xml version="1.0"?>
-<robot name="robot" xmlns:xacro="http://www.ros.org/wiki/xacro">
-    <xacro:include filename="$(find robot_description)/urdf/robot.gazebo" />
-    <!-- Parameters -->
-    <!-- pi already defined by default in xacro -->
-    <!-- <xacro:property name="pi" value="3.141592654" /> -->
-    <!-- Link - chassis-->
-    <link name="link_chassis">
-        <inertial>
-            <mass value="10" />
-            <origin xyz="0 0 0.3" rpy="0 0 0" />
-            <inertia ixx="1.5417" ixy="0" ixz="0" iyy="3.467" iyz="0" izz="4.742" />
-        </inertial>
-        <collision>
-            <geometry>
-                <box size="2 1.3 0.4" />
-            </geometry>
-        </collision>
-        <visual>
-            <geometry>
-                <box size="2 1.3 0.4" />
-            </geometry>
-            <material name="chassis_DarkBlue">
-                <color rgba="0 0 0.5 1" />
-            </material>
-        </visual>
-    </link>
-    <!-- Joint -chassis / left wheel-->
-    <joint name="joint_chassis_left_wheel" type="continuous">
-        <origin rpy="0 0 0" xyz="-0.5 0.65 0" />
-        <child link="link_left_wheel" />
-        <parent link="link_chassis" />
-        <axis rpy="0 0 0" xyz="0 1 0" />
-        <limit effort="1000" velocity="1000" />
-        <joint_properties damping="1.0" friction="1.0" />
-    </joint>
-    <!--Link - left wheel -->
-    <link name="link_left_wheel">
-        <inertial>
-            <mass value="1" />
-            <origin xyz="0 0 0" rpy="0 0 0" />
-            <inertia ixx="0.002526" ixy="0" ixz="0" iyy="0.002526" iyz="0" izz="0.005" />
-        </inertial>
-        <collision>
-            <origin rpy="${pi/2} 0 0" xyz="0 0.18 0" />
-            <geometry>
-                <cylinder length="0.12" radius="0.4" />
-            </geometry>
-        </collision>
-        <visual>
-            <origin rpy="${pi/2} 0 0" xyz="0 0.18 0" />
-            <geometry>
-                <cylinder length="0.12" radius="0.4" />
-            </geometry>
-            <material name="left_outer_black">
-                <color rgba="0 0 0 1" />
-            </material>
-        </visual>
-        <collision>
-            <origin rpy="${pi/2} 0 0" xyz="0 0.06 0" />
-            <geometry>
-                <cylinder length="0.12" radius="0.08" />
-            </geometry>
-        </collision>
-        <visual>
-            <origin rpy="${pi/2} 0 0" xyz="0 0.06 0" />
-            <geometry>
-                <cylinder length="0.12" radius="0.08" />
-            </geometry>
-            <material name="left_inner_black">
-                <color rgba="0 0 0 1" />
-            </material>
-        </visual>
-    </link>
-    <!-- Joint -chassis / right wheel-->
-    <joint name="joint_chassis_right_wheel" type="continuous">
-        <origin rpy="0 0 0" xyz="-0.5 -0.65 0" />
-        <child link="link_right_wheel" />
-        <parent link="link_chassis" />
-        <axis rpy="0 0 0" xyz="0 1 0" />
-        <limit effort="1000" velocity="1000" />
-        <joint_properties damping="1.0" friction="1.0" />
-    </joint>
-    <!--Link - right wheel -->
-    <link name="link_right_wheel">
-        <inertial>
-            <mass value="1" />
-            <origin xyz="0 0 0" rpy="0 0 0" />
-            <inertia ixx="0.002526" ixy="0" ixz="0" iyy="0.002526" iyz="0" izz="0.005" />
-        </inertial>
-        <collision>
-            <origin rpy="${pi/2} 0 0" xyz="0 -0.18 0" />
-            <geometry>
-                <cylinder length="0.12" radius="0.4" />
-            </geometry>
-        </collision>
-        <visual>
-            <origin rpy="${pi/2} 0 0" xyz="0 -0.18 0" />
-            <geometry>
-                <cylinder length="0.12" radius="0.4" />
-            </geometry>
-            <material name="right_outer_black">
-                <color rgba="0 0 0 1" />
-            </material>
-        </visual>
-        <collision>
-            <origin rpy="${pi/2} 0 0" xyz="0 -0.06 0" />
-            <geometry>
-                <cylinder length="0.12" radius="0.08" />
-            </geometry>
-        </collision>
-        <visual>
-            <origin rpy="${pi/2} 0 0" xyz="0 -0.06 0" />
-            <geometry>
-                <cylinder length="0.12" radius="0.08" />
-            </geometry>
-            <material name="right_inner_black">
-                <color rgba="0 0 0 1" />
-            </material>
-        </visual>
-    </link>
-    <!-- Joint -chassis / caster wheel-->
-    <joint name="joint_chassis_caster_wheel" type="fixed">
-        <origin rpy="0 0 0" xyz="0.8 0 -0.275" />
-        <child link="link_caster_wheel" />
-        <parent link="link_chassis" />
-    </joint>
-    <!--Link - caster wheel -->
-    <link name="link_caster_wheel">
-        <inertial>
-            <mass value="1" />
-            <origin xyz="0 0 0" rpy="0 0 0" />
-            <inertia ixx="0.0125" ixy="0" ixz="0" iyy="0.0125" iyz="0" izz="0.0125" />
-        </inertial>
-        <collision>
-            <origin rpy="0 0 0" xyz="0 0 0" />
-            <geometry>
-                <sphere radius="0.125" />
-            </geometry>
-        </collision>
-        <visual>
-            <origin rpy="0 0 0" xyz="0 0 0" />
-            <geometry>
-                <sphere radius="0.125" />
-            </geometry>
-            <material name="caster_darkblue">
-                <color rgba="0 0 0.5 1" />
-            </material>
-        </visual>
-    </link>
-    <!-- Laser Scan -->
-    <joint name="joint_laser_scan_chassis" type="fixed">
-        <origin rpy="0 0 0" xyz="0.8 0 0.3" />
-        <child link="link_laser_scan" />
-        <parent link="link_chassis" />
-        <joint_properties damping="1.0" friction="1.0" />
-    </joint>
-    <link name="link_laser_scan">
-        <inertial>
-            <origin rpy="0 0 0" xyz="0 0 0" />
-            <mass value="0.5" />
-            <inertia ixx="0.0002526" ixy="0" ixz="0" iyy="0.0002526" iyz="0" izz="0.0005" />
-        </inertial>
-        <visual>
-            <origin xyz="0 0 0" rpy="0 0 0" />
-            <geometry>
-                <cylinder radius="0.15" length="0.20" />
-            </geometry>
-            <material name="laser_scan_red">
-                <color rgba="0.7 0.1 0.1 1" />
-            </material>
-        </visual>
-        <collision>
-            <origin xyz="0 0 0" rpy="0 0 0" />
-            <geometry>
-                <cylinder radius="0.15" length="0.20" />
-            </geometry>
-        </collision>
-    </link>
-</robot>
+<xacro:root xmlns:xacro="http://www.ros.org/wiki/xacro">
+    <xacro:arg name="robot_name" default="my_robot"/>
+    <robot name="$(arg robot_name)">
+        <xacro:include filename="$(find robot_description)/urdf/robot.gazebo" />
+        <!-- Parameters -->
+        <!-- pi already defined by default in xacro -->
+        <!-- <xacro:property name="pi" value="3.141592654" /> -->
+        <!-- Link - chassis-->
+        <link name="link_chassis">
+            <inertial>
+                <mass value="10" />
+                <origin xyz="0 0 0.3" rpy="0 0 0" />
+                <inertia ixx="1.5417" ixy="0" ixz="0" iyy="3.467" iyz="0" izz="4.742" />
+            </inertial>
+            <collision>
+                <geometry>
+                    <box size="2 1.3 0.4" />
+                </geometry>
+            </collision>
+            <visual>
+                <geometry>
+                    <box size="2 1.3 0.4" />
+                </geometry>
+                <material name="chassis_DarkBlue">
+                    <color rgba="0 0 0.5 1" />
+                </material>
+            </visual>
+        </link>
+        <!-- Joint -chassis / left wheel -->
+        <joint name="joint_chassis_left_wheel" type="continuous">
+            <origin rpy="0 0 0" xyz="-0.5 0.65 0" />
+            <child link="link_left_wheel" />
+            <parent link="link_chassis" />
+            <axis rpy="0 0 0" xyz="0 1 0" />
+            <limit effort="1000" velocity="1000" />
+            <joint_properties damping="1.0" friction="1.0" />
+        </joint>
+        <!--Link - left wheel -->
+        <link name="link_left_wheel">
+            <inertial>
+                <mass value="1" />
+                <origin xyz="0 0 0" rpy="0 0 0" />
+                <inertia ixx="0.002526" ixy="0" ixz="0" iyy="0.002526" iyz="0" izz="0.005" />
+            </inertial>
+            <collision>
+                <origin rpy="${pi/2} 0 0" xyz="0 0.18 0" />
+                <geometry>
+                    <cylinder length="0.12" radius="0.4" />
+                </geometry>
+            </collision>
+            <visual>
+                <origin rpy="${pi/2} 0 0" xyz="0 0.18 0" />
+                <geometry>
+                    <cylinder length="0.12" radius="0.4" />
+                </geometry>
+                <material name="left_outer_black">
+                    <color rgba="0 0 0 1" />
+                </material>
+            </visual>
+            <collision>
+                <origin rpy="${pi/2} 0 0" xyz="0 0.06 0" />
+                <geometry>
+                    <cylinder length="0.12" radius="0.08" />
+                </geometry>
+            </collision>
+            <visual>
+                <origin rpy="${pi/2} 0 0" xyz="0 0.06 0" />
+                <geometry>
+                    <cylinder length="0.12" radius="0.08" />
+                </geometry>
+                <material name="left_inner_black">
+                    <color rgba="0 0 0 1" />
+                </material>
+            </visual>
+        </link>
+        <!-- Joint -chassis / right wheel-->
+        <joint name="joint_chassis_right_wheel" type="continuous">
+            <origin rpy="0 0 0" xyz="-0.5 -0.65 0" />
+            <child link="link_right_wheel" />
+            <parent link="link_chassis" />
+            <axis rpy="0 0 0" xyz="0 1 0" />
+            <limit effort="1000" velocity="1000" />
+            <joint_properties damping="1.0" friction="1.0" />
+        </joint>
+        <!--Link - right wheel -->
+        <link name="link_right_wheel">
+            <inertial>
+                <mass value="1" />
+                <origin xyz="0 0 0" rpy="0 0 0" />
+                <inertia ixx="0.002526" ixy="0" ixz="0" iyy="0.002526" iyz="0" izz="0.005" />
+            </inertial>
+            <collision>
+                <origin rpy="${pi/2} 0 0" xyz="0 -0.18 0" />
+                <geometry>
+                    <cylinder length="0.12" radius="0.4" />
+                </geometry>
+            </collision>
+            <visual>
+                <origin rpy="${pi/2} 0 0" xyz="0 -0.18 0" />
+                <geometry>
+                    <cylinder length="0.12" radius="0.4" />
+                </geometry>
+                <material name="right_outer_black">
+                    <color rgba="0 0 0 1" />
+                </material>
+            </visual>
+            <collision>
+                <origin rpy="${pi/2} 0 0" xyz="0 -0.06 0" />
+                <geometry>
+                    <cylinder length="0.12" radius="0.08" />
+                </geometry>
+            </collision>
+            <visual>
+                <origin rpy="${pi/2} 0 0" xyz="0 -0.06 0" />
+                <geometry>
+                    <cylinder length="0.12" radius="0.08" />
+                </geometry>
+                <material name="right_inner_black">
+                    <color rgba="0 0 0 1" />
+                </material>
+            </visual>
+        </link>
+        <!-- Joint -chassis / caster wheel-->
+        <joint name="joint_chassis_caster_wheel" type="fixed">
+            <origin rpy="0 0 0" xyz="0.8 0 -0.275" />
+            <child link="link_caster_wheel" />
+            <parent link="link_chassis" />
+        </joint>
+        <!--Link - caster wheel -->
+        <link name="link_caster_wheel">
+            <inertial>
+                <mass value="1" />
+                <origin xyz="0 0 0" rpy="0 0 0" />
+                <inertia ixx="0.0125" ixy="0" ixz="0" iyy="0.0125" iyz="0" izz="0.0125" />
+            </inertial>
+            <collision>
+                <origin rpy="0 0 0" xyz="0 0 0" />
+                <geometry>
+                    <sphere radius="0.125" />
+                </geometry>
+            </collision>
+            <visual>
+                <origin rpy="0 0 0" xyz="0 0 0" />
+                <geometry>
+                    <sphere radius="0.125" />
+                </geometry>
+                <material name="caster_darkblue">
+                    <color rgba="0 0 0.5 1" />
+                </material>
+            </visual>
+        </link>
+        <!-- Laser Scan -->
+        <joint name="joint_laser_scan_chassis" type="fixed">
+            <origin rpy="0 0 0" xyz="0.8 0 0.3" />
+            <child link="link_laser_scan" />
+            <parent link="link_chassis" />
+            <joint_properties damping="1.0" friction="1.0" />
+        </joint>
+        <link name="link_laser_scan">
+            <inertial>
+                <origin rpy="0 0 0" xyz="0 0 0" />
+                <mass value="0.5" />
+                <inertia ixx="0.0002526" ixy="0" ixz="0" iyy="0.0002526" iyz="0" izz="0.0005" />
+            </inertial>
+            <visual>
+                <origin xyz="0 0 0" rpy="0 0 0" />
+                <geometry>
+                    <cylinder radius="0.15" length="0.20" />
+                </geometry>
+                <material name="laser_scan_red">
+                    <color rgba="0.7 0.1 0.1 1" />
+                </material>
+            </visual>
+            <collision>
+                <origin xyz="0 0 0" rpy="0 0 0" />
+                <geometry>
+                    <cylinder radius="0.15" length="0.20" />
+                </geometry>
+            </collision>
+        </link>
+    </robot>
+</xacro:root>
